File: hw/led12/elec/layout/default/default.kicad_pcb (KiCad board)
At the start: 2 copper layers, 50 x 40 mm, 28 parts, among them Q1 Vgs ℝ+V, Q2 Vgs 1.75V

Commit message: hw: verified every part against the distributor
Checked all sixteen parts against LCSC product data and manufacturer
datasheets. Three of the parts chosen from memory were wrong for the job:

  - the bulk capacitor, Samsung CL32A107MQVNNNE, is a 6.3 V part, not 25 V.
    It would have failed on contact with a 12 V rail. 100 uF at 25 V does not
    exist in a 1210 MLCC at all; the largest purchasable is 47 uF, which is
    what the board now asks for.
  - the reverse-polarity P-FET, Si2301, is rated +/-8 V gate to source. This
    circuit holds its gate at ground while the source sits at the rail, so
    V_gs is the full 13.2 V in normal operation - not a surge case, the
    everyday one. Replaced with the AO3407A at +/-20 V, whose -30 V drain
    rating also clears the TVS clamping voltage that the Si2301's -20 V did
    not.
  - the fuse, 0466001.NR, is fast-acting: the 466 series is, despite the part
    having been picked to be slow-blow. Replaced with the 468 series, I2t
    0.127 A2s against 0.0423, so it survives inrush into the bulk cap.

Three more were real but poor choices: LCSC's Littelfuse SMBJ12A listing
carries SMBJ13A parameters, the LED's forward voltage was specified 1.6 to
2.6 V (too wide to size a resistor against), and the Alps switch and Phoenix
terminal were barely stocked and expensive respectively. All swapped for
parts that fit the same footprints.

Every supplier code has changed: the ones written from memory were guesses.

One finding is not yet addressed. The TVS clamps at 19.9 V while the LDO's
absolute maximum input is 15 V, so during a surge the regulator, not the TVS,
is the weakest part on the rail.

Co-Authored-By: Claude Opus 5 (1M context) <noreply@anthropic.com>
Parts:
- C1: value 100µF ±20% -> 47µF ±20%
Changed lines of the file:
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@@
 			)
 		)
-		(property "LCSC" "C471389"
+		(property "LCSC" "C8465"
 			(at 0 0 0)
 			(layer "User.9")
 			(hide yes)
 		)
-		(property "Manufacturer" "Phoenix Contact"
+		(property "Manufacturer" "Ningbo Kangnex"
 			(at 0 0 0)
 			(layer "User.9")
 			(hide yes)
 		)
-		(property "Partnumber" "1715721"
+		(property "Partnumber" "WJ500V-5.08-2P"
 			(at 0 0 0)
 			(layer "User.9")
@@
 			(hide yes)
 		)
-		(property "lcsc_id" "C471389"
+		(property "lcsc_id" "C8465"
 			(at 0 0 0)
 			(layer "User.9")
@@
 			)
 		)
-		(property "LCSC" "C881879"
+		(property "LCSC" "C45157"
 			(at 0 0 0)
 			(layer "User.9")
@@
 			(hide yes)
 		)
-		(property "Partnumber" "0466001.NR"
+		(property "Partnumber" "0468001.NRHF"
 			(at 0 0 0)
 			(layer "User.9")
@@
 			(hide yes)
 		)
-		(property "lcsc_id" "C881879"
+		(property "lcsc_id" "C45157"
 			(at 0 0 0)
 			(layer "User.9")
@@
 			)
 		)
-		(property "LCSC" "C10487"
+		(property "LCSC" "C15155"
 			(at 0 0 0)
 			(layer "User.9")
 			(hide yes)
 		)
-		(property "Manufacturer" "Vishay"
+		(property "Manufacturer" "Alpha & Omega Semiconductor"
 			(at 0 0 0)
 			(layer "User.9")
 			(hide yes)
 		)
-		(property "Partnumber" "SI2301CDS-T1-GE3"
+		(property "Partnumber" "AO3407A"
 			(at 0 0 0)
 			(layer "User.9")
@@
 			(hide yes)
 		)
-		(property "max_drain_source_voltage" "Vds max 20V"
+		(property "max_drain_source_voltage" "Vds max 30V"
 			(at 0 0 0)
 			(layer "User.9")
 			(hide yes)
 		)
-		(property "max_continuous_drain_current" "Id max 2.3A"
+		(property "max_continuous_drain_current" "Id max 4.3A"
 			(at 0 0 0)
 			(layer "User.9")
 			(hide yes)
 		)
-		(property "on_resistance" "Ron 100mΩ"
+		(property "on_resistance" "Ron 48mΩ"
 			(at 0 0 0)
 			(layer "User.9")
@@
 			(hide yes)
 		)
-		(property "lcsc_id" "C10487"
+		(property "lcsc_id" "C15155"
 			(at 0 0 0)
 			(layer "User.9")
@@
 			)
 		)
-		(property "LCSC" "C17407"
+		(property "LCSC" "C96346"
 			(at 0 0 0)
 			(layer "User.9")
@@
 			(hide yes)
 		)
-		(property "lcsc_id" "C17407"
+		(property "lcsc_id" "C96346"
 			(at 0 0 0)
 			(layer "User.9")
@@
 			)
 		)
-		(property "LCSC" "C908463"
+		(property "LCSC" "C111091"
 			(at 0 0 0)
 			(layer "User.9")
 			(hide yes)
 		)
-		(property "Manufacturer" "Littelfuse"
+		(property "Manufacturer" "Brightking"
 			(at 0 0 0)
 			(layer "User.9")
 			(hide yes)
 		)
-		(property "Partnumber" "SMBJ12A"
+		(property "Partnumber" "SMBJ12A/TR13"
 			(at 0 0 0)
 			(layer "User.9")
@@
 			(hide yes)
 		)
-		(property "lcsc_id" "C908463"
+		(property "lcsc_id" "C111091"
 			(at 0 0 0)
 			(layer "User.9")
@@
 			)
 		)
-		(property "Value" "100µF ±20%"
+		(property "Value" "47µF ±20%"
 			(at 0 2.3 0)
 			(layer "F.Fab")
@@
 			)
 		)
-		(property "LCSC" "C59461"
+		(property "LCSC" "C7432791"
 			(at 0 0 0)
 			(layer "User.9")
 			(hide yes)
 		)
-		(property "Manufacturer" "Samsung"
+		(property "Manufacturer" "Chinocera"
 			(at 0 0 0)
 			(layer "User.9")
 			(hide yes)
 		)
-		(property "Partnumber" "CL32A107MQVNNNE"
+		(property "Partnumber" "HGC1210R5476M250NSVK"
 			(at 0 0 0)
 			(layer "User.9")
 			(hide yes)
 		)
-		(property "capacitance" "100µF ±20%"
+		(property "capacitance" "47µF ±20%"
 			(at 0 0 0)
 			(layer "User.9")
@@
 			(hide yes)
 		)
-		(property "lcsc_id" "C59461"
+		(property "lcsc_id" "C7432791"
 			(at 0 0 0)
 			(layer "User.9")
@@
 			(hide yes)
 		)
-		(property "Manufacturer" "Samsung"
+		(property "Manufacturer" "YAGEO"
 			(at 0 0 0)
 			(layer "User.9")
 			(hide yes)
 		)
-		(property "Partnumber" "CL21B104KBCNNNC"
+		(property "Partnumber" "CC0805KRX7R9BB104"
 			(at 0 0 0)
 			(layer "User.9")
@@
 			)
 		)
-		(property "LCSC" "C115357"
+		(property "LCSC" "C110153"
 			(at 0 0 0)
 			(layer "User.9")
 			(hide yes)
 		)
-		(property "Manufacturer" "Alps"
+		(property "Manufacturer" "Korean Hroparts Elec"
 			(at 0 0 0)
 			(layer "User.9")
 			(hide yes)
 		)
-		(property "Partnumber" "SKHHAKA010"
+		(property "Partnumber" "K2-1102DP-C4SW-04"
 			(at 0 0 0)
 			(layer "User.9")
@@
 			(hide yes)
 		)
-		(property "lcsc_id" "C115357"
+		(property "lcsc_id" "C110153"
 			(at 0 0 0)
 			(layer "User.9")
@@
 			)
 		)
-		(property "LCSC" "C17414"
+		(property "LCSC" "C84376"
 			(at 0 0 0)
 			(layer "User.9")
@@
 			(hide yes)
 		)
-		(property "lcsc_id" "C17414"
+		(property "lcsc_id" "C84376"
 			(at 0 0 0)
 			(layer "User.9")
@@
 			)
 		)
-		(property "LCSC" "C17407"
+		(property "LCSC" "C96346"
 			(at 0 0 0)
 			(layer "User.9")
@@
 			(hide yes)
 		)
-		(property "lcsc_id" "C17407"
+		(property "lcsc_id" "C96346"
 			(at 0 0 0)
 			(layer "User.9")
@@
 			)
 		)
-		(property "LCSC" "C8545"
+		(property "LCSC" "C16338"
 			(at 0 0 0)
 			(layer "User.9")
@@
 			(hide yes)
 		)
-		(property "lcsc_id" "C8545"
+		(property "lcsc_id" "C16338"
 			(at 0 0 0)
 			(layer "User.9")
@@
 			(hide yes)
 		)
-		(property "Manufacturer" "Samsung"
+		(property "Manufacturer" "YAGEO"
 			(at 0 0 0)
 			(layer "User.9")
 			(hide yes)
 		)
-		(property "Partnumber" "CL21B104KBCNNNC"
+		(property "Partnumber" "CC0805KRX7R9BB104"
 			(at 0 0 0)
 			(layer "User.9")
@@
 			)
 		)
-		(property "LCSC" "C96446"
+		(property "LCSC" "C15850"
 			(at 0 0 0)
 			(layer "User.9")
@@
 			(hide yes)
 		)
-		(property "lcsc_id" "C96446"
+		(property "lcsc_id" "C15850"
 			(at 0 0 0)
 			(layer "User.9")
@@
 			)
 		)
-		(property "LCSC" "C17568"
+		(property "LCSC" "C114531"
 			(at 0 0 0)
 			(layer "User.9")
@@
 			(hide yes)
 		)
-		(property "lcsc_id" "C17568"
+		(property "lcsc_id" "C114531"
 			(at 0 0 0)
 			(layer "User.9")
@@
 			)
 		)
-		(property "LCSC" "C17673"
+		(property "LCSC" "C114549"
 			(at 0 0 0)
 			(layer "User.9")
@@
 			(hide yes)
 		)
-		(property "lcsc_id" "C17673"
+		(property "lcsc_id" "C114549"
 			(at 0 0 0)
 			(layer "User.9")
@@
 			)
 		)
-		(property "LCSC" "C72038"
+		(property "LCSC" "C2943978"
 			(at 0 0 0)
 			(layer "User.9")
@@
 			(hide yes)
 		)
-		(property "Partnumber" "19-217/R6C-AL1M2VY/3T"
+		(property "Partnumber" "17-21SURC/S530-A3/4T"
 			(at 0 0 0)
 			(layer "User.9")
@@
 			(hide yes)
 		)
-		(property "lcsc_id" "C72038"
+		(property "lcsc_id" "C2943978"
 			(at 0 0 0)
 			(layer "User.9")
@@
 			)
 		)
-		(property "LCSC" "C17673"
+		(property "LCSC" "C114549"
 			(at 0 0 0)
 			(layer "User.9")
@@
 			(hide yes)
 		)
-		(property "lcsc_id" "C17673"
+		(property "lcsc_id" "C114549"
 			(at 0 0 0)
 			(layer "User.9")
@@
 			)
 		)
-		(property "LCSC" "C72038"
+		(property "LCSC" "C2943978"
 			(at 0 0 0)
 			(layer "User.9")
@@
 			(hide yes)
 		)
-		(property "Partnumber" "19-217/R6C-AL1M2VY/3T"
+		(property "Partnumber" "17-21SURC/S530-A3/4T"
 			(at 0 0 0)
 			(layer "User.9")
@@
 			(hide yes)
 		)
-		(property "lcsc_id" "C72038"
+		(property "lcsc_id" "C2943978"
 			(at 0 0 0)
 			(layer "User.9")
@@
 			)
 		)
-		(property "LCSC" "C17673"
+		(property "LCSC" "C114549"
 			(at 0 0 0)
 			(layer "User.9")
@@
 			(hide yes)
 		)
-		(property "lcsc_id" "C17673"
+		(property "lcsc_id" "C114549"
 			(at 0 0 0)
 			(layer "User.9")
@@
 			)
 		)
-		(property "LCSC" "C72038"
+		(property "LCSC" "C2943978"
 			(at 0 0 0)
 			(layer "User.9")
@@
 			(hide yes)
 		)
-		(property "Partnumber" "19-217/R6C-AL1M2VY/3T"
+		(property "Partnumber" "17-21SURC/S530-A3/4T"
 			(at 0 0 0)
 			(layer "User.9")
@@
 			(hide yes)
 		)
-		(property "lcsc_id" "C72038"
+		(property "lcsc_id" "C2943978"
 			(at 0 0 0)
 			(layer "User.9")
@@
 			)
 		)
-		(property "LCSC" "C17673"
+		(property "LCSC" "C114549"
 			(at 0 0 0)
 			(layer "User.9")
@@
 			(hide yes)
 		)
-		(property "lcsc_id" "C17673"
+		(property "lcsc_id" "C114549"
 			(at 0 0 0)
 			(layer "User.9")
@@
 			)
 		)
-		(property "LCSC" "C72038"
+		(property "LCSC" "C2943978"
 			(at 0 0 0)
 			(layer "User.9")
@@
 			(hide yes)
 		)
-		(property "Partnumber" "19-217/R6C-AL1M2VY/3T"
+		(property "Partnumber" "17-21SURC/S530-A3/4T"
 			(at 0 0 0)
 			(layer "User.9")
@@
 			(hide yes)
 		)
-		(property "lcsc_id" "C72038"
+		(property "lcsc_id" "C2943978"
 			(at 0 0 0)
 			(layer "User.9")

Commit message: hw: electrical and topology checks, and the two defects they found
Eighteen more checks, in three tiers, all reading values out of the build
rather than restating them.

test_electrical.py does the arithmetic atopile structurally cannot: LED current
across the supply range, resistor dissipation against rating, gate drive against
the FET threshold, debounce time constants, fuse headroom, and whether anything
on the protected rail is rated below what the TVS lets through. Corners are
taken from each declared range, so narrowing a tolerance moves the result
without editing a check.

test_topology.py verifies the shape those computations assume - that the fuse
really is first, that nothing bypasses the reverse-polarity FET, that each LED
has its own resistor, that every rail has a test point, and that the 12 V net
reaches exactly the parts the electrical checks apply the rail voltage to.

They found two real defects on first run.

The LED series resistors were 680 R, carried over from a 5 V way of thinking.
On a 12 V rail the LED drops 2.2 V and the resistor takes the other 9.8, so at
13.8 mA it dissipated 130 mW in a 125 mW part: 104 % of rating at nominal and
137 % at the corner. Now 2.2 k, giving 3.7 to 5.1 mA at 45 % of rating. Keeping
10 mA would have meant a 1206 resistor and a second package on the board, which
is not worth it for an indicator.

The regulator was rated 15 V against a TVS that clamps at 19.9 V, so the part
the protection exists to protect was the first thing a surge would destroy. That
is not fixable at the TVS end - a device standing off 13.2 V cannot clamp below
15 V - so the regulator moved. The Gainsil GS2401C-33 survives 44 V and operates
to 40 V, so a clamp event leaves it inside its normal range. Its quiescent
current is 1.3 uA against about 5 mA, which on this board is most of the idle
draw, and it costs slightly less than a genuine AMS1117. Its input capacitor
went to 1 uF, which is what its datasheet characterises.

That pinout is rare: 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
Parts:
- C3: value 100nF ±10% -> 1µF ±10%
- R1, R2, R3, R4: value 680Ω ±1% -> 2.2kΩ ±1%
Changed lines of the file:
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@@
 			(hide yes)
 		)
-		(property "on_resistance" "Ron ℝ+Ω"
+		(property "on_resistance" "Ron 7.5Ω"
 			(at 0 0 0)
 			(layer "User.9")
@@
 			)
 		)
-		(property "LCSC" "C6186"
-			(at 0 0 0)
-			(layer "User.9")
-			(hide yes)
-		)
-		(property "Manufacturer" "Advanced Monolithic Systems"
-			(at 0 0 0)
-			(layer "User.9")
-			(hide yes)
-		)
-		(property "Partnumber" "AMS1117-3.3"
+		(property "LCSC" "C6283798"
+			(at 0 0 0)
+			(layer "User.9")
+			(hide yes)
+		)
+		(property "Manufacturer" "Gainsil"
+			(at 0 0 0)
+			(layer "User.9")
+			(hide yes)
+		)
+		(property "Partnumber" "GS2401C-33CTR3"
 			(at 0 0 0)
 			(layer "User.9")
@@
 			(hide yes)
 		)
-		(property "lcsc_id" "C6186"
+		(property "lcsc_id" "C6283798"
 			(at 0 0 0)
 			(layer "User.9")
@@
 			)
 		)
-		(property "Value" "100nF ±10%"
+		(property "Value" "1µF ±10%"
 			(at 0 1.68 0)
 			(layer "F.Fab")
@@
 			)
 		)
-		(property "LCSC" "C49678"
-			(at 0 0 0)
-			(layer "User.9")
-			(hide yes)
-		)
-		(property "Manufacturer" "YAGEO"
-			(at 0 0 0)
-			(layer "User.9")
-			(hide yes)
-		)
-		(property "Partnumber" "CC0805KRX7R9BB104"
-			(at 0 0 0)
-			(layer "User.9")
-			(hide yes)
-		)
-		(property "capacitance" "100nF ±10%"
+		(property "LCSC" "C28323"
+			(at 0 0 0)
+			(layer "User.9")
+			(hide yes)
+		)
+		(property "Manufacturer" "Samsung"
+			(at 0 0 0)
+			(layer "User.9")
+			(hide yes)
+		)
+		(property "Partnumber" "CL21B105KBFNNNE"
+			(at 0 0 0)
+			(layer "User.9")
+			(hide yes)
+		)
+		(property "capacitance" "1µF ±10%"
 			(at 0 0 0)
 			(layer "User.9")
@@
 			(hide yes)
 		)
-		(property "lcsc_id" "C49678"
+		(property "lcsc_id" "C28323"
 			(at 0 0 0)
 			(layer "User.9")
@@
 			)
 		)
-		(property "Value" "680Ω ±1%"
+		(property "Value" "2.2kΩ ±1%"
 			(at 0 1.65 0)
 			(layer "F.Fab")
@@
 			)
 		)
-		(property "LCSC" "C114549"
+		(property "LCSC" "C114561"
 			(at 0 0 0)
 			(layer "User.9")
@@
 			(hide yes)
 		)
-		(property "Partnumber" "RC0805FR-07680RL"
-			(at 0 0 0)
-			(layer "User.9")
-			(hide yes)
-		)
-		(property "resistance" "680Ω ±1%"
+		(property "Partnumber" "RC0805FR-072K2L"
+			(at 0 0 0)
+			(layer "User.9")
+			(hide yes)
+		)
+		(property "resistance" "2.2kΩ ±1%"
 			(at 0 0 0)
 			(layer "User.9")
@@
 			(hide yes)
 		)
-		(property "lcsc_id" "C114549"
+		(property "lcsc_id" "C114561"
 			(at 0 0 0)
 			(layer "User.9")
@@
 			)
 		)
-		(property "Value" "680Ω ±1%"
+		(property "Value" "2.2kΩ ±1%"
 			(at 0 1.65 0)
 			(layer "F.Fab")
@@
 			)
 		)
-		(property "LCSC" "C114549"
+		(property "LCSC" "C114561"
 			(at 0 0 0)
 			(layer "User.9")
@@
 			(hide yes)
 		)
-		(property "Partnumber" "RC0805FR-07680RL"
-			(at 0 0 0)
-			(layer "User.9")
-			(hide yes)
-		)
-		(property "resistance" "680Ω ±1%"
+		(property "Partnumber" "RC0805FR-072K2L"
+			(at 0 0 0)
+			(layer "User.9")
+			(hide yes)
+		)
+		(property "resistance" "2.2kΩ ±1%"
 			(at 0 0 0)
 			(layer "User.9")
@@
 			(hide yes)
 		)
-		(property "lcsc_id" "C114549"
+		(property "lcsc_id" "C114561"
 			(at 0 0 0)
 			(layer "User.9")
@@
 			)
 		)
-		(property "Value" "680Ω ±1%"
+		(property "Value" "2.2kΩ ±1%"
 			(at 0 1.65 0)
 			(layer "F.Fab")
@@
 			)
 		)
-		(property "LCSC" "C114549"
+		(property "LCSC" "C114561"
 			(at 0 0 0)
 			(layer "User.9")
@@
 			(hide yes)
 		)
-		(property "Partnumber" "RC0805FR-07680RL"
-			(at 0 0 0)
-			(layer "User.9")
-			(hide yes)
-		)
-		(property "resistance" "680Ω ±1%"
+		(property "Partnumber" "RC0805FR-072K2L"
+			(at 0 0 0)
+			(layer "User.9")
+			(hide yes)
+		)
+		(property "resistance" "2.2kΩ ±1%"
 			(at 0 0 0)
 			(layer "User.9")
@@
 			(hide yes)
 		)
-		(property "lcsc_id" "C114549"
+		(property "lcsc_id" "C114561"
 			(at 0 0 0)
 			(layer "User.9")
@@
 			)
 		)
-		(property "Value" "680Ω ±1%"
+		(property "Value" "2.2kΩ ±1%"
 			(at 0 1.65 0)
 			(layer "F.Fab")
@@
 			)
 		)
-		(property "LCSC" "C114549"
+		(property "LCSC" "C114561"
 			(at 0 0 0)
 			(layer "User.9")
@@
 			(hide yes)
 		)
-		(property "Partnumber" "RC0805FR-07680RL"
-			(at 0 0 0)
-			(layer "User.9")
-			(hide yes)
-		)
-		(property "resistance" "680Ω ±1%"
+		(property "Partnumber" "RC0805FR-072K2L"
+			(at 0 0 0)
+			(layer "User.9")
+			(hide yes)
+		)
+		(property "resistance" "2.2kΩ ±1%"
 			(at 0 0 0)
 			(layer "User.9")
@@
 			(hide yes)
 		)
-		(property "lcsc_id" "C114549"
-			(at 0 0 0)
-			(layer "User.9")
+		(property "lcsc_id" "C114561"
+			(at 0 0 0)
+			(layer "User.9")
