File: hw/led12/elec/layout/default/default.kicad_pcb (KiCad board)
At the start: 2 copper layers, 50 x 40 mm, 28 parts, among them Q1 Vgs ℝ+V, Q2 Vgs 1.75V

Commit message: hw: place and route the board, and the bug that fell out of it
The board is now laid out: 28 parts placed, 63 track segments, 12 stitching
vias and a ground pour on the back copper. KiCad DRC reports nothing at any
severity - no shorts, nothing unconnected, no silkscreen over a pad - against
both the PCBWay limits and the board's own rules.

Placement and routing are data, in led12/layout.py, applied by tools/layout.py.
Routes name pads symbolically - "power.q_rpp:3" is that FET's drain - so moving
a part in the placement table moves the tracks that reach it, and literal
coordinates are only the corners in between. The engine refuses to run unless
every part on the board is placed deliberately, so a part added upstream cannot
quietly land at the origin.

Two properties make it safe on every build. It is idempotent: everything it
writes carries a recognisable UUID prefix and is removed before being written
again, so positions come from the description and never from accumulated edits.
And it is deterministic: UUIDs are derived from what the object is, so a
rebuild that changes nothing produces no diff.

Laying it out found a real circuit bug that every earlier check had passed.
atopile's `~>` bridges a diode from anode to cathode, so `out.hv ~> tvs ~>
out.lv` reads perfectly and puts the protection device across the rail
backwards, where it conducts at 0.7 V and shorts the supply. DRC caught it as a
short between 12V and GND. The connection is now written by name, and
test_polarised_parts_face_the_right_way checks every polarised pin against the
net its datasheet expects - the earlier topology checks only asked which parts
were on a net, never which pin.

Zone filling needs KiCad's own Python module. kicad-cli cannot fill, and it
runs DRC against whatever fill is in the file, so an unfilled plane reports
every ground pad as unconnected while looking fine.

Silkscreen took several passes. atopile puts each designator on top of the part
it names, which the fab clips aw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
Parts:
- moved TP3 276.2 mm to (-6.00, 10.0)
- moved TP4 249.0 mm to (11.0, -2.00)
- moved TP1 230.5 mm to (19.5, -2.00)
- moved TP2 224.5 mm to (15.5, -2.00)
- moved D4 224.5 mm to (6.00, 15.0)
- moved R4 208.5 mm to (12.0, 15.0), turned to 180 degrees
- moved D3 204.3 mm to (6.00, 11.0)
- moved R3 188.3 mm to (12.0, 11.0), turned to 180 degrees
- moved D2 184.1 mm to (6.00, 7.00)
- moved R2 168.1 mm to (12.0, 7.00), turned to 180 degrees
- moved D1 164.0 mm to (6.00, 3.00)
- moved R1 148.0 mm to (12.0, 3.00), turned to 180 degrees
- moved R6 130.6 mm to (19.5, -5.00)
- moved C4 120.8 mm to (19.5, -8.00)
- moved C3 118.7 mm to (11.5, -6.00)
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Connections:
- D5 pad 1: GND -> 12V
- D5 pad 2: 12V -> GND
Routing:
- net 12V: track 0.00 -> 127.6 mm
- net GND: track 0.00 -> 27.5 mm, vias 0 -> 12
- net LED_RETURN: track 0.00 -> 23.3 mm
- net 3V3: track 0.00 -> 21.3 mm
- net VIN_RAW: track 0.00 -> 16.7 mm
- net GATE: track 0.00 -> 15.2 mm
- net RPP_GATE: track 0.00 -> 10.1 mm
- net BTN: track 0.00 -> 10.1 mm
- net leds[3]-LED_A: track 0.00 -> 4.15 mm
- net leds[2]-LED_A: track 0.00 -> 4.15 mm
- net leds[1]-LED_A: track 0.00 -> 4.15 mm
- net LED_A: track 0.00 -> 4.15 mm
- net VIN_FUSED: track 0.00 -> 3.21 mm
- added copper zone on B.Cu, net GND
